Commit message: base_link joint is actually a base_footprint.

File: ev3infoumons_ros/ev3infoumons_description/urdf/ev3infoumons.urdf (robot description, URDF)
Before this commit: robot ev3infoumons, 2 links, 1 joints
Links:
- removed link base_link
- added link base_footprint; visual mesh filename=package://ev3infoumons_description/meshes/base_pivoted.dae
Joints:
- removed joint base_link_to_base_laser
- added joint base_footprint_to_base_laser: type fixed, parent base_footprint, child base_laser, origin xyz=0.02 0 0.095
